File: ESPHomeACMonitor.kicad_pcb (KiCad board)
At the start: 2 copper layers, 45 x 78 mm, 26 parts, among them J1 DEBUG, J2 T/C_1, J3 T/C_2, J4 24VAC_SUPPLY, SW1 RESET, U1 ESP32-WROVER-E, U2 XGZP6899D, U3 MAX31855KASA, U4 MAX31855KASA, U5 LM2576S-3.3

Commit message: Added 3D Models
Parts:
- U2: footprint Sensor_Pressure:CFSensor_XGZP6899x -> ESPHomeACMonitor:XGZP6899x
- moved U2 0.50 mm to (66.0, 93.5)
